Commit message: Add exercice3

File: exercice3/simple_pendulum.urdf (robot description, URDF)
Before this commit: robot pendulum, 5 links, 4 joints
Links:
- removed link SecondPendulumArm
- removed link SecondPendulumMass
- link PendulumArm: geometry visual box size=0.01 0.01 1.0
- link PendulumMass: mass 300.0 -> 10.0
- link world: mass 0.0 -> 1000.0
Joints:
- removed joint SecondPendulumJoint
- removed joint SecondPendulumMassJoint
- joint PendulumMassJoint: origin xyz=0.0 0.0 0.5 rpy=0 0 0 -> xyz=0.0 0.0 1.0 rpy=0 0 0
